File: arm/sch/datalogger_arm.sch (KiCad schematic (older format))
At the start: 24 parts

Commit message: More work on arm board. going to add RF in place of SD
Parts:
- removed IC?: MCP73831T, symbol MCP73831T
- removed IC?: MCP1802T-3002I-OT, symbol MCP1802T-3002I-OT
- removed IC?: MCP102T-315ETT, symbol MCP102T-315ETT
- added C? (x2): 4.7u, symbol C
- added IC?: MCP1603T, symbol MCP1603T
- added IC?: MCP102T-315ETT, symbol MCP102T-315ETT
- added L?: 4.7u, symbol INDUCTOR
- added P?: BAT, symbol CONN_2
- added Q?: BSH121, symbol BSH121
- added R? (x3): 10k, symbol R
- added SW?: SWITCH_INV_MECH, symbol SWITCH_INV_MECH
Connections:
- net labels added: +3.3V, A0, A1, A2, A3, CHECK_BAT, HALF_BAT, I2C_SCL, I2C_SDA, PWRA, PWRB
- wire segments 88 -> 128
- no-connect marks 1 -> 2
Other:
- moved on the sheet: C?, IC?, P?, R?, SW?, X?
